File: gear-display/PCB/GDBM/level_shifter.kicad_sch (KiCad schematic)
At the start: 3 parts

Commit message: updates
Connections:
- net +3V3: no longer names the net of C?.1, U?.1 (VCC)
Changed lines of the file:
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@@
     (pin "9")
-  )
-  (symbol (lib_id "power:+3V3") (at 148.59 55.88 0) (unit 1)
-    (in_bom yes) (on_board yes) (fields_autoplaced)
-    (property "Reference" "#PWR?" (id 0) (at 148.59 59.69 0)
-      (effects (font (size 1.27 1.27)) hide)
-    )
-    (property "Value" "+3V3" (id 1) (at 148.59 50.8 0))
-    (property "Footprint" "" (id 2) (at 148.59 55.88 0)
-      (effects (font (size 1.27 1.27)) hide)
-    )
-    (property "Datasheet" "" (id 3) (at 148.59 55.88 0)
-      (effects (font (size 1.27 1.27)) hide)
-    )
-    (pin "1")
   )
   (symbol (lib_id "power:GND") (at 137.16 72.39 0) (unit 1)
