File: gear-display/PCB/GDBM/GDBM.kicad_sch (KiCad schematic)
At the start: 2 parts, among them J1 Con_Screw_1x04_691313510004, J2 Con_Screw_1x04_691313510004

Commit message: layout
Connections:
- no-connect marks 10 -> 11
Other:
- sheet Brightness Control ports: added none; removed POT_W
