File: gear-display/PCB/GDBM/GDBM.kicad_sch (KiCad schematic)
At the start: 2 parts, among them J1 Con_Screw_1x04_691313510004, J2 Con_Screw_1x04_691313510004

Commit message: R33 value change
Parts:
- added R31: R_0402_4700_1%, KD_Resistor:RESC1005X40N, symbol KD_Resistor:R_0402_4700_1%
Connections:
- net 7-Segment Display/PWM: now also R31.2
- new net MCU/A5(D23): R31.1
Changed lines of the file:
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@@
+    (stroke (width 0) (type default))
+  )
+  (wire (pts (xy 81.28 55.88) (xy 100.33 55.88))
     (stroke (width 0) (type default))
   )
@@
     (stroke (width 0) (type default))
   )
+  (wire (pts (xy 107.95 55.88) (xy 133.35 55.88))
+    (stroke (width 0) (type default))
+  )
   (wire (pts (xy 205.74 91.44) (xy 213.36 91.44))
     (stroke (width 0) (type default))
@@
   )
   (wire (pts (xy 205.74 104.14) (xy 213.36 104.14))
-    (stroke (width 0) (type default))
-  )
-  (wire (pts (xy 133.35 55.88) (xy 81.28 55.88))
     (stroke (width 0) (type default))
   )
@@
         )
       )
+    )
+  )
+  (symbol (lib_id "KD_Resistor:R_0402_4700_1%") (at 104.14 55.88 90) (unit 1)
+    (in_bom yes) (on_board yes) (dnp no) (fields_autoplaced)
+    (property "Reference" "R31" (at 104.14 50.8 90)
+      (effects (font (size 1.27 1.27)))
+    )
+    (property "Value" "R_0402_4700_1%" (at 72.39 68.58 0)
+      (effects (font (size 1.27 1.27)) (justify left) hide)
+    )
+    (property "Footprint" "KD_Resistor:RESC1005X40N" (at 90.17 68.58 0)
+      (effects (font (size 1.27 1.27)) (justify left) hide)
+    )
+    (property "Datasheet" "https://www.te.com/commerce/DocumentDelivery/DDEController?Action=srchrtrv&DocNm=1773204-3&DocType=DS&DocLang=English" (at 92.71 68.58 0)
+      (effects (font (size 1.27 1.27)) (justify left) hide)
+    )
+    (property "Code" "4k7" (at 104.14 53.34 90)
+      (effects (font (size 1.27 1.27)))
+    )
+    (property "Manufacturer" "Bourns Inc." (at 74.93 68.58 0)
+      (effects (font (size 1.27 1.27)) (justify left) hide)
+    )
+    (property "MFG_PartNo" "CR0402-FX-4701GLF" (at 77.47 68.58 0)
+      (effects (font (size 1.27 1.27)) (justify left) hide)
+    )
+    (property "Supplier" "Digi-Key" (at 80.01 68.58 0)
+      (effects (font (size 1.27 1.27)) (justify left) hide)
+    )
+    (property "Supplier_PartNo" "CR0402-FX-4701GLFCT-ND" (at 82.55 68.58 0)
+      (effects (font (size 1.27 1.27)) (justify left) hide)
+    )
+    (property "DNP" "F" (at 85.09 68.58 0)
+      (effects (font (size 1.27 1.27)) (justify left) hide)
+    )
+    (property "Price" "0.01" (at 87.63 68.58 0)
+      (effects (font (size 1.27 1.27)) (justify left) hide)
+    )
+    (pin "1")
+    (pin "2")
+    (instances
+      (project "GDBM"
+        (path "/e63e39d7-6ac0-4ffd-8aa3-1841a4541b55/d5432ca7-524c-447e-b53c-48db40cafebb"
+          (reference "R31") (unit 1)
+        )
+        (path "/e63e39d7-6ac0-4ffd-8aa3-1841a4541b55"
+          (reference "R34") (unit 1)
+        )
+      )

Commit message: version numbering fix
Changed lines of the file:
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@@
   (title_block
     (title "Gear Display Board")
-    (date "2023-04-06")
-    (rev "3.0")
+    (date "2023-09-22")
+    (rev "4.0")
     (company "Kallio Designs Oy")
     (comment 1 "Teemu Latonen")
@@
     )
   )
-  (sheet (at 39.37 74.93) (size 25.4 12.7) (fields_autoplaced)
-    (stroke (width 0.1524) (type solid))
-    (fill (color 0 0 0 0.0000))
-    (property "Sheetname" "Revision History" (at 39.37 74.2184 0)
-      (effects (font (size 1.27 1.27)) (justify left bottom))
-    )
-    (property "Sheetfile" "rev_history.kicad_sch" (at 39.37 88.2146 0)
+  (sheet (at 39.37 83.82) (size 25.4 12.7) (fields_autoplaced)
+    (stroke (width 0.1524) (type solid))
+    (fill (color 0 0 0 0.0000))
+    (property "Sheetname" "Revision History" (at 39.37 83.1084 0)
+      (effects (font (size 1.27 1.27)) (justify left bottom))
+    )
+    (property "Sheetfile" "rev_history.kicad_sch" (at 39.37 97.1046 0)
       (effects (font (size 1.27 1.27)) (justify left top))
     )
@@
     )
   )
-  (sheet (at 39.37 54.61) (size 25.4 12.7) (fields_autoplaced)
-    (stroke (width 0.1524) (type solid))
-    (fill (color 0 0 0 0.0000))
-    (property "Sheetname" "Mechanical" (at 39.37 53.8984 0)
-      (effects (font (size 1.27 1.27)) (justify left bottom))
-    )
-    (property "Sheetfile" "mechanical.kicad_sch" (at 39.37 67.8946 0)
+  (sheet (at 39.37 63.5) (size 25.4 12.7) (fields_autoplaced)
+    (stroke (width 0.1524) (type solid))
+    (fill (color 0 0 0 0.0000))
+    (property "Sheetname" "Mechanical" (at 39.37 62.7884 0)
+      (effects (font (size 1.27 1.27)) (justify left bottom))
+    )
+    (property "Sheetfile" "mechanical.kicad_sch" (at 39.37 76.7846 0)
       (effects (font (size 1.27 1.27)) (justify left top))
     )
@@
     )
   )
-  (sheet (at 39.37 34.29) (size 25.4 12.7) (fields_autoplaced)
-    (stroke (width 0.1524) (type solid))
-    (fill (color 0 0 0 0.0000))
-    (property "Sheetname" "Power Supply" (at 39.37 33.5784 0)
-      (effects (font (size 1.27 1.27)) (justify left bottom))
-    )
-    (property "Sheetfile" "psu.kicad_sch" (at 39.37 47.5746 0)
-      (effects (font (size 1.27 1.27)) (justify left top))
-    )
+  (sheet (at 39.37 43.18) (size 25.4 12.7) (fields_autoplaced)
+    (stroke (width 0.1524) (type solid))
+    (fill (color 0 0 0 0.0000))
+    (property "Sheetname" "Power Supply" (at 39.37 42.4684 0)
+      (effects (font (size 1.27 1.27)) (justify left bottom))
+    )
+    (property "Sheetfile" "psu.kicad_sch" (at 39.37 56.4646 0)
+      (effects (font (size 1.27 1.27)) (justify left top))
+    )

Commit message: Layout
Parts:
- J1, J2: value Con_Screw_1x04_691313510004 -> 1x04
- R31: value R_0402_4700_1% -> 4k7
Changed lines of the file:
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@@
       (effects (font (size 1.27 1.27)))
     )
-    (property "Value" "Con_Screw_1x04_691313510004" (at 250.19 195.58 0)
+    (property "Value" "1x04" (at 250.19 195.58 0)
       (effects (font (size 1.27 1.27)) (justify left) hide)
     )
@@
       (effects (font (size 1.27 1.27)))
     )
-    (property "Value" "R_0402_4700_1%" (at 72.39 68.58 0)
+    (property "Value" "4k7" (at 72.39 68.58 0)
       (effects (font (size 1.27 1.27)) (justify left) hide)
     )
@@
       (effects (font (size 1.27 1.27)))
     )
-    (property "Value" "Con_Screw_1x04_691313510004" (at 60.96 196.85 0)
+    (property "Value" "1x04" (at 60.96 196.85 0)
       (effects (font (size 1.27 1.27)) (justify left) hide)
     )

Commit message: Documentation and version update
Parts:
- renumbered R31 to R34
