File: gear-display/PCB/GDBM/indicators.kicad_sch (KiCad schematic)
At the start: 4 parts

Commit message: rikki
Parts:
- R23, R24, R25: renamed from R?; footprint KD_Resistor:R_0805_2012Metric -> KD_Resistor:RESC2012X60N
- gave numbers to parts that had none: 1
Connections:
- net B renamed INDICATOR_B
- net G renamed INDICATOR_G
- net R renamed INDICATOR_R
Other:
- company: (none) -> Kallio Designs Oy
- title: (none) -> Gear Display Board
Changed lines of the file:
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@@
 (kicad_sch (version 20211123) (generator eeschema)
   (paper "A4")
+  (title_block
+    (title "Gear Display Board")
+    (date "2022-08-13")
+    (rev "1.0")
+    (company "Kallio Designs Oy")
+    (comment 1 "Teemu Latonen")
+    (comment 2 "000064")
+    (comment 3 "000065")
+  )
   (wire (pts (xy 129.54 105.41) (xy 129.54 99.06))
     (stroke (width 0) (type default) (color 0 0 0 0))
@@
     (effects (font (size 1.27 1.27)) (justify left bottom))
   )
-  (hierarchical_label "R" (shape input) (at 87.63 105.41 180)
+  (hierarchical_label "INDICATOR_R" (shape input) (at 87.63 105.41 180)
     (effects (font (size 1.27 1.27)) (justify right))
   )
-  (hierarchical_label "G" (shape input) (at 87.63 111.76 180)
+  (hierarchical_label "INDICATOR_G" (shape input) (at 87.63 111.76 180)
     (effects (font (size 1.27 1.27)) (justify right))
   )
-  (hierarchical_label "B" (shape input) (at 87.63 118.11 180)
+  (hierarchical_label "INDICATOR_B" (shape input) (at 87.63 118.11 180)
     (effects (font (size 1.27 1.27)) (justify right))
   )
@@
   (symbol (lib_id "KD_Resistor:R_0805_0_automotive") (at 129.54 95.25 0) (unit 1)
     (in_bom yes) (on_board yes) (fields_autoplaced)
-    (property "Reference" "R?" (id 0) (at 132.08 93.9799 0)
+    (property "Reference" "R23" (id 0) (at 132.08 93.9799 0)
       (effects (font (size 1.27 1.27)) (justify left))
     )
@@
       (effects (font (size 1.27 1.27)) (justify left) hide)
     )
-    (property "Footprint" "KD_Resistor:R_0805_2012Metric" (id 2) (at 116.84 81.28 0)
+    (property "Footprint" "KD_Resistor:RESC2012X60N" (id 2) (at 116.84 81.28 0)
       (effects (font (size 1.27 1.27)) (justify left) hide)
     )
@@
   (symbol (lib_id "KD_Resistor:R_0805_0_automotive") (at 139.7 95.25 0) (unit 1)
     (in_bom yes) (on_board yes) (fields_autoplaced)
-    (property "Reference" "R?" (id 0) (at 142.24 93.9799 0)
+    (property "Reference" "R24" (id 0) (at 142.24 93.9799 0)
       (effects (font (size 1.27 1.27)) (justify left))
     )
@@
       (effects (font (size 1.27 1.27)) (justify left) hide)
     )
-    (property "Footprint" "KD_Resistor:R_0805_2012Metric" (id 2) (at 127 81.28 0)
+    (property "Footprint" "KD_Resistor:RESC2012X60N" (id 2) (at 127 81.28 0)
       (effects (font (size 1.27 1.27)) (justify left) hide)
     )
@@
   (symbol (lib_id "KD_Resistor:R_0805_0_automotive") (at 149.86 95.25 0) (unit 1)
     (in_bom yes) (on_board yes) (fields_autoplaced)
-    (property "Reference" "R?" (id 0) (at 152.4 93.9799 0)
+    (property "Reference" "R25" (id 0) (at 152.4 93.9799 0)
       (effects (font (size 1.27 1.27)) (justify left))
     )
@@
       (effects (font (size 1.27 1.27)) (justify left) hide)
     )
-    (property "Footprint" "KD_Resistor:R_0805_2012Metric" (id 2) (at 137.16 81.28 0)
+    (property "Footprint" "KD_Resistor:RESC2012X60N" (id 2) (at 137.16 81.28 0)
       (effects (font (size 1.27 1.27)) (justify left) hide)
     )
@@
   (symbol (lib_id "KD_Connector_Screw:Con_Screw_1x04_691313510004") (at 157.48 77.47 0) (unit 1)
     (in_bom yes) (on_board yes) (fields_autoplaced)
-    (property "Reference" "J?" (id 0) (at 165.1 80.0099 0)
+    (property "Reference" "J5" (id 0) (at 165.1 80.0099 0)
       (effects (font (size 1.27 1.27)) (justify left))
     )

Commit message: PSU and LED powering changed
Connections:
- net 12V_PWM: now also J5.4 (Pin_4); no longer J5.1 (Pin_1)
- net at J5.2 (Pin_2): now also R24.1; no longer R23.1
- net at J5.3 (Pin_3): now also R23.1; no longer R24.1
- net at R25.1: now also J5.1 (Pin_1); no longer J5.4 (Pin_4)
Other:
- note removed: "Shift indicator"
Changed lines of the file:
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@@
     (stroke (width 0) (type default) (color 0 0 0 0))
-  )
-  (text "Shift indicator" (at 149.86 72.39 0)
-    (effects (font (size 1.27 1.27)) (justify left bottom))
   )
   (hierarchical_label "INDICATOR_R" (shape input) (at 87.63 105.41 180)
@@
   (hierarchical_label "12V_PWM" (shape input) (at 87.63 77.47 180)
     (effects (font (size 1.27 1.27)) (justify right))
+  )
+  (symbol (lib_id "KD_Connector_Screw:Con_Screw_1x04_691313510004") (at 157.48 85.09 0) (mirror x) (unit 1)
+    (in_bom yes) (on_board yes) (fields_autoplaced)
+    (property "Reference" "J5" (id 0) (at 162.56 71.12 0))
+    (property "Value" "Con_Screw_1x04_691313510004" (id 1) (at 144.78 116.84 0)
+      (effects (font (size 1.27 1.27)) (justify left) hide)
+    )
+    (property "Footprint" "KD_Connector_Screw:CON_508_1X04_691313510004_Mated" (id 2) (at 144.78 99.06 0)
+      (effects (font (size 1.27 1.27)) (justify left) hide)
+    )
+    (property "Datasheet" "https://www.we-online.com/katalog/datasheet/6913135100xx.pdf" (id 3) (at 144.78 96.52 0)
+      (effects (font (size 1.27 1.27)) (justify left) hide)
+    )
+    (property "Code" "1x04" (id 4) (at 162.56 73.66 0))
+    (property "Manufacturer" "Würth Elektronik" (id 5) (at 144.78 114.3 0)
+      (effects (font (size 1.27 1.27)) (justify left) hide)
+    )
+    (property "MFG_PartNo" "691313510004" (id 6) (at 144.78 111.76 0)
+      (effects (font (size 1.27 1.27)) (justify left) hide)
+    )
+    (property "Supplier" "Digi-Key" (id 7) (at 144.78 109.22 0)
+      (effects (font (size 1.27 1.27)) (justify left) hide)
+    )
+    (property "Supplier_PartNo" "732-2072-ND" (id 8) (at 144.78 106.68 0)
+      (effects (font (size 1.27 1.27)) (justify left) hide)
+    )
+    (property "DNP" "F" (id 9) (at 144.78 104.14 0)
+      (effects (font (size 1.27 1.27)) (justify left) hide)
+    )
+    (property "Price" "0.3" (id 10) (at 144.78 101.6 0)
+      (effects (font (size 1.27 1.27)) (justify left) hide)
+    )
+    (pin "1")
+    (pin "2")
+    (pin "3")
+    (pin "4")
   )
   (symbol (lib_id "KD_Resistor:R_0805_0_automotive") (at 129.54 95.25 0) (unit 1)
@@
     (pin "2")
   )
-  (symbol (lib_id "KD_Connector_Screw:Con_Screw_1x04_691313510004") (at 157.48 77.47 0) (unit 1)
-    (in_bom yes) (on_board yes) (fields_autoplaced)
-    (property "Reference" "J5" (id 0) (at 165.1 80.0099 0)
-      (effects (font (size 1.27 1.27)) (justify left))
-    )
-    (property "Value" "Con_Screw_1x04_691313510004" (id 1) (at 144.78 45.72 0)
-      (effects (font (size 1.27 1.27)) (justify left) hide)
-    )
-    (property "Footprint" "KD_Connector_Screw:CON_508_1X04_691313510004_Mated" (id 2) (at 144.78 63.5 0)
-      (effects (font (size 1.27 1.27)) (justify left) hide)
-    )
-    (property "Datasheet" "https://www.we-online.com/katalog/datasheet/6913135100xx.pdf" (id 3) (at 144.78 66.04 0)
-      (effects (font (size 1.27 1.27)) (justify left) hide)
-    )
-    (property "Code" "1x04" (id 4) (at 165.1 82.5499 0)
-      (effects (font (size 1.27 1.27)) (justify left))
-    )
-    (property "Manufacturer" "Würth Elektronik" (id 5) (at 144.78 48.26 0)
-      (effects (font (size 1.27 1.27)) (justify left) hide)
-    )
-    (property "MFG_PartNo" "691313510004" (id 6) (at 144.78 50.8 0)
-      (effects (font (size 1.27 1.27)) (justify left) hide)
-    )
-    (property "Supplier" "Digi-Key" (id 7) (at 144.78 53.34 0)
-      (effects (font (size 1.27 1.27)) (justify left) hide)
-    )
-    (property "Supplier_PartNo" "732-2072-ND" (id 8) (at 144.78 55.88 0)
-      (effects (font (size 1.27 1.27)) (justify left) hide)
-    )
-    (property "DNP" "F" (id 9) (at 144.78 58.42 0)
-      (effects (font (size 1.27 1.27)) (justify left) hide)
-    )
-    (property "Price" "0.3" (id 10) (at 144.78 60.96 0)
-      (effects (font (size 1.27 1.27)) (justify left) hide)
-    )
-    (pin "1")
-    (pin "2")
-    (pin "3")
-    (pin "4")
-  )
 )
