File: gear-display/PCB/GDBM/indicators.kicad_sch (KiCad schematic)
At the start: 4 parts, among them J5 Con_Screw_1x04_691313510004

Commit message: Layout
Parts:
- J5: value Con_Screw_1x04_691313510004 -> 1x04
- R23, R24, R25: value R_0805_0_automotive -> 0; symbol KD_Resistor:R_0805_0_automotive -> KD_Resistor:R_0805_0
Changed lines of the file:
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@@
       (effects (font (size 1.27 1.27)))
     )
-    (property "Value" "Con_Screw_1x04_691313510004" (at 144.78 116.84 0)
+    (property "Value" "1x04" (at 144.78 116.84 0)
       (effects (font (size 1.27 1.27)) (justify left) hide)
     )
@@
     )
   )
-  (symbol (lib_id "KD_Resistor:R_0805_0_automotive") (at 129.54 95.25 0) (unit 1)
+  (symbol (lib_id "KD_Resistor:R_0805_0") (at 129.54 95.25 0) (unit 1)
     (in_bom yes) (on_board yes) (dnp no) (fields_autoplaced)
-    (property "Reference" "R23" (at 132.08 93.9799 0)
+    (property "Reference" "R23" (at 132.08 93.98 0)
       (effects (font (size 1.27 1.27)) (justify left))
     )
-    (property "Value" "R_0805_0_automotive" (at 116.84 63.5 0)
+    (property "Value" "0" (at 116.84 63.5 0)
       (effects (font (size 1.27 1.27)) (justify left) hide)
     )
@@
       (effects (font (size 1.27 1.27)) (justify left) hide)
     )
-    (property "Code" "0" (at 132.08 96.5199 0)
+    (property "Code" "0" (at 132.08 96.52 0)
       (effects (font (size 1.27 1.27)) (justify left))
     )
@@
     )
   )
-  (symbol (lib_id "KD_Resistor:R_0805_0_automotive") (at 139.7 95.25 0) (unit 1)
+  (symbol (lib_id "KD_Resistor:R_0805_0") (at 139.7 95.25 0) (unit 1)
     (in_bom yes) (on_board yes) (dnp no) (fields_autoplaced)
-    (property "Reference" "R24" (at 142.24 93.9799 0)
+    (property "Reference" "R24" (at 142.24 93.98 0)
       (effects (font (size 1.27 1.27)) (justify left))
     )
-    (property "Value" "R_0805_0_automotive" (at 127 63.5 0)
+    (property "Value" "0" (at 127 63.5 0)
       (effects (font (size 1.27 1.27)) (justify left) hide)
     )
@@
       (effects (font (size 1.27 1.27)) (justify left) hide)
     )
-    (property "Code" "0" (at 142.24 96.5199 0)
+    (property "Code" "0" (at 142.24 96.52 0)
       (effects (font (size 1.27 1.27)) (justify left))
     )
@@
     )
   )
-  (symbol (lib_id "KD_Resistor:R_0805_0_automotive") (at 149.86 95.25 0) (unit 1)
+  (symbol (lib_id "KD_Resistor:R_0805_0") (at 149.86 95.25 0) (unit 1)
     (in_bom yes) (on_board yes) (dnp no) (fields_autoplaced)
-    (property "Reference" "R25" (at 152.4 93.9799 0)
+    (property "Reference" "R25" (at 152.4 93.98 0)
       (effects (font (size 1.27 1.27)) (justify left))
     )
-    (property "Value" "R_0805_0_automotive" (at 137.16 63.5 0)
+    (property "Value" "0" (at 137.16 63.5 0)
       (effects (font (size 1.27 1.27)) (justify left) hide)
     )
@@
       (effects (font (size 1.27 1.27)) (justify left) hide)
     )
-    (property "Code" "0" (at 152.4 96.5199 0)
+    (property "Code" "0" (at 152.4 96.52 0)
       (effects (font (size 1.27 1.27)) (justify left))
     )
