File: gear-display/PCB/GDBM/usb.kicad_sch (KiCad schematic)
At the start: 7 parts

Commit message: updates
Parts:
- removed C?: C_0805_1u_X7R_25V, KD_Capacitor:C_0805_2012Metric, symbol KD_Capacitor:C_0805_1u_X7R_25V
- added C?: C_1206_10u_50V, KD_Capacitor:C_1206_3216Metric, symbol KD_Capacitor:C_1206_10u_50V
- X?: symbol KD_Connector_USB_HDMI_Etc:USB_MiniB_V_651005136421 -> KD_Connector_USB_HDMI_Etc:USB_B_V_Adam_USB-B-S-VT; MFG_PartNo 651005136421 -> USB-B-S-VT; Manufacturer Wurth Elektronik -> Adam Tech; Price 3 -> 1; Supplier_PartNo 732-2735-ND -> 2057-USB-B-S-VT-ND
Connections:
- net GND: now also X?.4 (GND), C?.2; no longer X?.GND
- net USB_CON_D_N: now also X?.2 (D-); no longer X?.D-
- net USB_CON_D_P: now also X?.3 (D+); no longer X?.D+
- net USB_VBUS: now also C?.1
- net at D?.5 (V+), FB?.1: now also X?.1 (VBUS); no longer X?.VBUS
- no-connect marks 1 -> 0
Other:
- moved on the sheet: C?

Commit message: changed to match simhub conf
Changed lines of the file:
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@@
     (stroke (width 0) (type default) (color 0 0 0 0))
-  )
-  (label "USB_VBUS" (at 152.4 62.23 180)
-    (effects (font (size 1.27 1.27)) (justify right bottom))
   )
   (label "USB_CON_D_N" (at 105.41 99.06 180)
@@
     (effects (font (size 1.27 1.27)) (justify left))
   )
+  (hierarchical_label "USB_VBUS" (shape output) (at 152.4 62.23 0)
+    (effects (font (size 1.27 1.27)) (justify left))
+  )

Commit message: rikki
Parts:
- removed X?: USB_MiniB_V_651005136421, KD_Connector_USB_HDMI_Etc:CON_USB-MINIB_651005136421, symbol KD_Connector_USB_HDMI_Etc:USB_B_V_Adam_USB-B-S-VT
- added J8: USB_B_V_Adam_USB-B-S-VT, KD_Connector_USB_HDMI_Etc:USB_B_Vertical_Adam_USB-B-S-VT, symbol KD_Connector_USB_HDMI_Etc:USB_B_V_Adam_USB-B-S-VT
- R10, R9: renamed from R?; footprint KD_Resistor:R_0603_1608Metric -> KD_Resistor:RESC1608X55N
- gave numbers to parts that had none: 4
Connections:
- net Earth: now also J8.H1 (Shield), J8.H2 (Shield)
- net GND: now also J8.4 (GND)
- net USB_CON_D_N: now also J8.2 (D-)
- net USB_CON_D_P: now also J8.3 (D+)
- net at D4.5 (V+), FB1.1: now also J8.1 (VBUS)
- no-connect marks 0 -> 2
Changed lines of the file:
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@@
   (title_block
     (title "Gear Display Board")
-    (date "2022-08-07")
+    (date "2022-08-13")
     (rev "1.0")
     (company "Kallio Designs Oy")
     (comment 1 "Teemu Latonen")
-    (comment 2 "ASSEMBLY_PN")
-    (comment 3 "PCB_PN")
-  )
+    (comment 2 "000064")
+    (comment 3 "000065")
+  )
+  (bus_alias "USB" (members "USB_CON_D_P" "USB_CON_D_N"))
   (junction (at 91.44 99.06) (diameter 0) (color 0 0 0 0)
   )
@@
   (junction (at 88.9 91.44) (diameter 0) (color 0 0 0 0)
   )
+  (no_connect (at 92.71 144.78))
+  (no_connect (at 107.95 144.78))
   (wire (pts (xy 110.49 62.23) (xy 110.49 64.77))
     (stroke (width 0) (type default) (color 0 0 0 0))
@@
   (symbol (lib_id "power:GND") (at 110.49 74.93 0) (unit 1)
     (in_bom yes) (on_board yes)
-    (property "Reference" "#PWR?" (id 0) (at 110.49 81.28 0)
+    (property "Reference" "#PWR0115" (id 0) (at 110.49 81.28 0)
       (effects (font (size 1.27 1.27)) hide)
     )
@@
   (symbol (lib_id "KD_Inductor:Ferrite_250mA_Murata_BLM15HG102SN1D") (at 102.87 62.23 90) (unit 1)
     (in_bom yes) (on_board yes) (fields_autoplaced)
-    (property "Reference" "FB?" (id 0) (at 102.87 55.88 90))
+    (property "Reference" "FB1" (id 0) (at 102.87 55.88 90))
     (property "Value" "Ferrite_250mA_Murata_BLM15HG102SN1D" (id 1) (at 71.12 74.93 0)
       (effects (font (size 1.27 1.27)) (justify left) hide)
@@
     (pin "2")
   )
+  (symbol (lib_id "KD_Resistor:R_0603_10_5%") (at 120.65 102.87 90) (unit 1)
+    (in_bom yes) (on_board yes) (fields_autoplaced)
+    (property "Reference" "R10" (id 0) (at 120.65 96.52 90))
+    (property "Value" "R_0603_10_5%" (id 1) (at 88.9 115.57 0)
+      (effects (font (size 1.27 1.27)) (justify left) hide)
+    )
+    (property "Footprint" "KD_Resistor:RESC1608X55N" (id 2) (at 106.68 115.57 0)
+      (effects (font (size 1.27 1.27)) (justify left) hide)
+    )
+    (property "Datasheet" "https://www.te.com/commerce/DocumentDelivery/DDEController?Action=srchrtrv&DocNm=1773204-3&DocType=DS&DocLang=English" (id 3) (at 109.22 115.57 0)
+      (effects (font (size 1.27 1.27)) (justify left) hide)
+    )
+    (property "Code" "10" (id 4) (at 120.65 99.06 90))
+    (property "Manufacturer" "Walsin Technology Corporation" (id 5) (at 91.44 115.57 0)
+      (effects (font (size 1.27 1.27)) (justify left) hide)
+    )
+    (property "MFG_PartNo" "WR06X100 JTL" (id 6) (at 93.98 115.57 0)
+      (effects (font (size 1.27 1.27)) (justify left) hide)
+    )
+    (property "Supplier" "Digi-Key" (id 7) (at 96.52 115.57 0)
+      (effects (font (size 1.27 1.27)) (justify left) hide)
+    )
+    (property "Supplier_PartNo" "1292-WR06X100JTLCT-ND" (id 8) (at 99.06 115.57 0)
+      (effects (font (size 1.27 1.27)) (justify left) hide)
+    )
+    (property "DNP" "F" (id 9) (at 101.6 115.57 0)
+      (effects (font (size 1.27 1.27)) (justify left) hide)
+    )
+    (property "Price" "0.01" (id 10) (at 104.14 115.57 0)
+      (effects (font (size 1.27 1.27)) (justify left) hide)
+    )
+    (pin "1")
+    (pin "2")
+  )
   (symbol (lib_id "KD_Connector_USB_HDMI_Etc:USB_B_V_Adam_USB-B-S-VT") (at 76.2 96.52 0) (unit 1)
     (in_bom yes) (on_board yes) (fields_autoplaced)
-    (property "Reference" "X?" (id 0) (at 76.2 83.82 0))
-    (property "Value" "USB_MiniB_V_651005136421" (id 1) (at 68.58 60.96 0)
-      (effects (font (size 1.27 1.27)) (justify left) hide)
-    )
-    (property "Footprint" "KD_Connector_USB_HDMI_Etc:CON_USB-MINIB_651005136421" (id 2) (at 68.58 78.74 0)
+    (property "Reference" "J8" (id 0) (at 76.2 83.82 0))
+    (property "Value" "USB_B_V_Adam_USB-B-S-VT" (id 1) (at 68.58 60.96 0)
+      (effects (font (size 1.27 1.27)) (justify left) hide)
+    )
+    (property "Footprint" "KD_Connector_USB_HDMI_Etc:USB_B_Vertical_Adam_USB-B-S-VT" (id 2) (at 68.58 78.74 0)
       (effects (font (size 1.27 1.27)) (justify left) hide)
     )
@@
       (effects (font (size 1.27 1.27)) (justify left) hide)
     )
-    (property "Code" "USB Mini B" (id 4) (at 68.326 87.503 0)
-      (effects (font (size 1.27 1.27)) (justify left))
-    )
+    (property "Code" "USB Mini B" (id 4) (at 76.2 86.36 0))
     (property "Manufacturer" "Adam Tech" (id 5) (at 68.58 63.5 0)
       (effects (font (size 1.27 1.27)) (justify left) hide)
@@
     (pin "H2")
   )
-  (symbol (lib_id "KD_Resistor:R_0603_10_5%") (at 120.65 102.87 90) (unit 1)
-    (in_bom yes) (on_board yes) (fields_autoplaced)
-    (property "Reference" "R?" (id 0) (at 120.65 96.52 90))
-    (property "Value" "R_0603_10_5%" (id 1) (at 88.9 115.57 0)
-      (effects (font (size 1.27 1.27)) (justify left) hide)
-    )
-    (property "Footprint" "KD_Resistor:R_0603_1608Metric" (id 2) (at 106.68 115.57 0)
-      (effects (font (size 1.27 1.27)) (justify left) hide)
-    )
-    (property "Datasheet" "https://www.te.com/commerce/DocumentDelivery/DDEController?Action=srchrtrv&DocNm=1773204-3&DocType=DS&DocLang=English" (id 3) (at 109.22 115.57 0)
-      (effects (font (size 1.27 1.27)) (justify left) hide)
-    )
-    (property "Code" "10" (id 4) (at 120.65 99.06 90))
-    (property "Manufacturer" "Walsin Technology Corporation" (id 5) (at 91.44 115.57 0)
-      (effects (font (size 1.27 1.27)) (justify left) hide)
-    )
-    (property "MFG_PartNo" "WR06X100 JTL" (id 6) (at 93.98 115.57 0)
-      (effects (font (size 1.27 1.27)) (justify left) hide)
-    )
-    (property "Supplier" "Digi-Key" (id 7) (at 96.52 115.57 0)
-      (effects (font (size 1.27 1.27)) (justify left) hide)
-    )
-    (property "Supplier_PartNo" "1292-WR06X100JTLCT-ND" (id 8) (at 99.06 115.57 0)
-      (effects (font (size 1.27 1.27)) (justify left) hide)
-    )
-    (property "DNP" "F" (id 9) (at 101.6 115.57 0)
-      (effects (font (size 1.27 1.27)) (justify left) hide)
-    )
-    (property "Price" "0.01" (id 10) (at 104.14 115.57 0)
-      (effects (font (size 1.27 1.27)) (justify left) hide)
-    )
-    (pin "1")
-    (pin "2")
-  )
   (symbol (lib_id "KD_Capacitor:C_1206_10u_50V") (at 110.49 68.58 0) (unit 1)
     (in_bom yes) (on_board yes) (fields_autoplaced)
-    (property "Reference" "C?" (id 0) (at 114.3 67.3099 0)
+    (property "Reference" "C12" (id 0) (at 114.3 67.3099 0)
       (effects (font (size 1.27 1.27)) (justify left))
     )
@@
   (symbol (lib_id "power:GND") (at 121.92 140.97 0) (unit 1)
     (in_bom yes) (on_board yes)
-    (property "Reference" "#PWR?" (id 0) (at 121.92 147.32 0)
+    (property "Reference" "#PWR0114" (id 0) (at 121.92 147.32 0)
       (effects (font (size 1.27 1.27)) hide)
     )
@@
   (symbol (lib_id "KD_Capacitor:C_0603_100n_X7R_100V") (at 127 68.58 0) (unit 1)
     (in_bom yes) (on_board yes) (fields_autoplaced)
-    (property "Reference" "C?" (id 0) (at 130.81 67.3099 0)
+    (property "Reference" "C13" (id 0) (at 130.81 67.3099 0)
       (effects (font (size 1.27 1.27)) (justify left))
     )
@@
   (symbol (lib_id "power:Earth") (at 71.12 115.57 0) (unit 1)
     (in_bom yes) (on_board yes) (fields_autoplaced)
-    (property "Reference" "#PWR?" (id 0) (at 71.12 121.92 0)
+    (property "Reference" "#PWR0112" (id 0) (at 71.12 121.92 0)
       (effects (font (size 1.27 1.27)) hide)
     )
@@
   (symbol (lib_id "KD_Diode:TVS_5V5_DRTR5V0U4S-7-M") (at 100.33 137.16 0) (unit 1)
     (in_bom yes) (on_board yes) (fields_autoplaced)
-    (property "Reference" "D?" (id 0) (at 100.33 123.19 0))
+    (property "Reference" "D4" (id 0) (at 100.33 123.19 0))
     (property "Value" "TVS_5V5_DRTR5V0U4S-7-M" (id 1) (at 85.09 92.71 0)
       (effects (font (size 1.27 1.27)) (justify left) hide)
@@
   (symbol (lib_id "power:GND") (at 127 74.93 0) (unit 1)
     (in_bom yes) (on_board yes)
-    (property "Reference" "#PWR?" (id 0) (at 127 81.28 0)
+    (property "Reference" "#PWR0116" (id 0) (at 127 81.28 0)
       (effects (font (size 1.27 1.27)) hide)
     )
@@
   (symbol (lib_id "KD_Resistor:R_0603_10_5%") (at 120.65 92.71 90) (unit 1)
     (in_bom yes) (on_board yes) (fields_autoplaced)
-    (property "Reference" "R?" (id 0) (at 120.65 86.36 90))
+    (property "Reference" "R9" (id 0) (at 120.65 86.36 90))
     (property "Value" "R_0603_10_5%" (id 1) (at 88.9 105.41 0)
       (effects (font (size 1.27 1.27)) (justify left) hide)
     )
-    (property "Footprint" "KD_Resistor:R_0603_1608Metric" (id 2) (at 106.68 105.41 0)
+    (property "Footprint" "KD_Resistor:RESC1608X55N" (id 2) (at 106.68 105.41 0)
       (effects (font (size 1.27 1.27)) (justify left) hide)
     )
@@
   (symbol (lib_id "power:GND") (at 76.2 115.57 0) (unit 1)
     (in_bom yes) (on_board yes)
-    (property "Reference" "#PWR?" (id 0) (at 76.2 121.92 0)
-      (effects (font (size 1.27 1.27)) hide)
-    )
+    (property "Reference" "#PWR0113" (id 0) (at 76.2 121.92 0)
+      (effects (font (size 1.27 1.27)) hide)
+    )

Commit message: PSU and LED powering changed
Parts:
- C12: footprint KD_Capacitor:C_1206_3216Metric -> KD_Capacitor:CAPC3216X150N
- C13: footprint KD_Capacitor:C_0603_1608Metric -> KD_Capacitor:CAPC1608X90N
Changed lines of the file:
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@@
       (effects (font (size 1.27 1.27)) (justify left) hide)
     )
-    (property "Footprint" "KD_Capacitor:C_1206_3216Metric" (id 2) (at 97.79 54.61 0)
+    (property "Footprint" "KD_Capacitor:CAPC3216X150N" (id 2) (at 97.79 54.61 0)
       (effects (font (size 1.27 1.27)) (justify left) hide)
     )
@@
       (effects (font (size 1.27 1.27)) (justify left) hide)
     )
-    (property "Footprint" "KD_Capacitor:C_0603_1608Metric" (id 2) (at 114.3 54.61 0)
+    (property "Footprint" "KD_Capacitor:CAPC1608X90N" (id 2) (at 114.3 54.61 0)
       (effects (font (size 1.27 1.27)) (justify left) hide)
     )

Commit message: layout
Parts:
- C12: value C_1206_10u_50V -> C_1206_10u_X5R_50V_automotive; symbol KD_Capacitor:C_1206_10u_50V -> KD_Capacitor:C_1206_10u_X5R_50V_automotive; Code 10 uF -> 10u; MFG_PartNo CL31B106KBHNNNE -> GRT31CR61H106ME01L; Manufacturer Samsung Electro-Mechanics -> Murata Electronics; Price 0.10 -> 0.30; Supplier_PartNo 1276-6767-1-ND -> 490-12457-1-ND
Changed lines of the file:
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@@
   (title_block
     (title "Gear Display Board")
-    (date "2022-08-13")
-    (rev "1.0")
+    (date "2023-01-05")
+    (rev "2.0")
     (company "Kallio Designs Oy")
     (comment 1 "Teemu Latonen")
@@
     (pin "H2")
   )
-  (symbol (lib_id "KD_Capacitor:C_1206_10u_50V") (at 110.49 68.58 0) (unit 1)
+  (symbol (lib_id "KD_Capacitor:C_1206_10u_X5R_50V_automotive") (at 110.49 68.58 0) (unit 1)
     (in_bom yes) (on_board yes) (fields_autoplaced)
     (property "Reference" "C12" (id 0) (at 114.3 67.3099 0)
       (effects (font (size 1.27 1.27)) (justify left))
     )
-    (property "Value" "C_1206_10u_50V" (id 1) (at 97.79 36.83 0)
+    (property "Value" "C_1206_10u_X5R_50V_automotive" (id 1) (at 97.79 36.83 0)
       (effects (font (size 1.27 1.27)) (justify left) hide)
     )
@@
       (effects (font (size 1.27 1.27)) (justify left) hide)
     )
-    (property "Datasheet" "datasheet" (id 3) (at 97.79 57.15 0)
-      (effects (font (size 1.27 1.27)) (justify left) hide)
-    )
-    (property "Code" "10 uF" (id 4) (at 114.3 69.8499 0)
+    (property "Datasheet" "https://search.murata.co.jp/Ceramy/image/img/A01X/G101/ENG/GRT31CR61H106ME01-01.pdf" (id 3) (at 97.79 57.15 0)
+      (effects (font (size 1.27 1.27)) (justify left) hide)
+    )
+    (property "Code" "10u" (id 4) (at 114.3 69.8499 0)
       (effects (font (size 1.27 1.27)) (justify left))
     )
-    (property "Manufacturer" "Samsung Electro-Mechanics" (id 5) (at 97.79 39.37 0)
-      (effects (font (size 1.27 1.27)) (justify left) hide)
-    )
-    (property "MFG_PartNo" "CL31B106KBHNNNE" (id 6) (at 97.79 41.91 0)
+    (property "Manufacturer" "Murata Electronics" (id 5) (at 97.79 39.37 0)
+      (effects (font (size 1.27 1.27)) (justify left) hide)
+    )
+    (property "MFG_PartNo" "GRT31CR61H106ME01L" (id 6) (at 97.79 41.91 0)
       (effects (font (size 1.27 1.27)) (justify left) hide)
     )
@@
       (effects (font (size 1.27 1.27)) (justify left) hide)
     )
-    (property "Supplier_PartNo" "1276-6767-1-ND" (id 8) (at 97.79 46.99 0)
+    (property "Supplier_PartNo" "490-12457-1-ND" (id 8) (at 97.79 46.99 0)
       (effects (font (size 1.27 1.27)) (justify left) hide)
     )
@@
       (effects (font (size 1.27 1.27)) (justify left) hide)
     )
-    (property "Price" "0.10" (id 10) (at 97.79 52.07 0)
-      (effects (font (size 1.27 1.27)) (justify left) hide)
-    )
+    (property "Price" "0.30" (id 10) (at 97.79 52.07 0)
+      (effects (font (size 1.27 1.27)) (justify left) hide)
+    )
