File: gear-display/PCB/GDBM/usb.kicad_sch (KiCad schematic)
At the start: 7 parts, among them J8 USB_B_V_Adam_USB-B-S-VT

Commit message: Layout
Parts:
- C12: value C_1206_10u_X5R_50V_automotive -> 10u
- C13: value C_0603_100n_X7R_100V -> 100n
- J8: value USB_B_V_Adam_USB-B-S-VT -> USB Mini B
Changed lines of the file:
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@@
       (effects (font (size 1.27 1.27)))
     )
-    (property "Value" "USB_B_V_Adam_USB-B-S-VT" (at 68.58 60.96 0)
+    (property "Value" "USB Mini B" (at 68.58 60.96 0)
       (effects (font (size 1.27 1.27)) (justify left) hide)
     )
@@
       (effects (font (size 1.27 1.27)) (justify left))
     )
-    (property "Value" "C_1206_10u_X5R_50V_automotive" (at 97.79 36.83 0)
+    (property "Value" "10u" (at 97.79 36.83 0)
       (effects (font (size 1.27 1.27)) (justify left) hide)
     )
@@
       (effects (font (size 1.27 1.27)) (justify left))
     )
-    (property "Value" "C_0603_100n_X7R_100V" (at 114.3 36.83 0)
+    (property "Value" "100n" (at 114.3 36.83 0)
       (effects (font (size 1.27 1.27)) (justify left) hide)
     )
