File: gear-display/PCB/GDBM/rev_history.kicad_sch (KiCad schematic)
At the start: 0 parts

Commit message: updates
Other:
- note added: "Reversed R28 potentiometer action"
Changed lines of the file:
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@@
+    (stroke (width 0) (type solid) (color 0 0 0 1))
+  )
+  (polyline (pts (xy 57.15 114.3) (xy 243.84 114.3))
     (stroke (width 0) (type solid) (color 0 0 0 1))
   )
@@
     (effects (font (size 3 3) (thickness 1) bold) (justify left bottom))
   )
+  (text "Reversed R28 potentiometer action" (at 90.17 111.76 0)
+    (effects (font (size 2 2)) (justify left bottom))
+  )
   (text "R33 changed to 110 ohm for brightness scaling" (at 90.17 104.14 0)
