File: gear-display/PCB/GDBM/rev_history.kicad_sch (KiCad schematic)
At the start: 0 parts

Commit message: version numbering fix
Other:
- note added: "4.00"
- note added: "C22 Updated"
Changed lines of the file:
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@@
   (title_block
     (title "Gear Display Board")
-    (date "2023-04-06")
-    (rev "3.0")
+    (date "2023-09-22")
+    (rev "4.0")
     (company "Kallio Designs Oy")
     (comment 1 "Teemu Latonen")
@@
     (effects (font (size 2 2)) (justify left bottom))
   )
+  (text "27.03.2023" (at 69.85 111.76 0)
+    (effects (font (size 2 2)) (justify left bottom))
+  )
+  (text "C22 Updated" (at 90.17 111.76 0)
+    (effects (font (size 2 2)) (justify left bottom))
+  )
+  (text "4.00" (at 59.69 111.76 0)
+    (effects (font (size 2 2)) (justify left bottom))
+  )

Commit message: Layout
Changed lines of the file:
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@@
+    (effects (font (size 2 2)) (justify left bottom))
+  )
+  (text "Teemu Latonen" (at 208.28 111.76 0)
     (effects (font (size 2 2)) (justify left bottom))
   )
