File: gear-display/PCB/GDBM/led_driver.kicad_sch (KiCad schematic)
At the start: 5 parts

Commit message: new features
Connections:
- net +3V3 renamed +5V
Changed lines of the file:
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@@
   )
   (bus_alias "I2C" (members "SDA" "SCL"))
-  (bus_alias "SPI" (members "MISO" "MOSI" "SCL"))
+  (bus_alias "SPI" (members "MISO" "MOSI" "SCLK"))
   (junction (at 163.83 63.5) (diameter 0) (color 0 0 0 0)
   )
@@
   (hierarchical_label "SRCK" (shape input) (at 120.65 100.33 180)
     (effects (font (size 1.27 1.27)) (justify right))
-  )
-  (symbol (lib_id "power:+3V3") (at 163.83 57.15 0)
-    (in_bom yes) (on_board yes) (fields_autoplaced)
-    (property "Reference" "#PWR?" (id 0) (at 163.83 60.96 0)
-      (effects (font (size 1.27 1.27)) hide)
-    )
-    (property "Value" "+3V3" (id 1) (at 163.83 52.07 0))
-    (property "Footprint" "" (id 2) (at 163.83 57.15 0)
-      (effects (font (size 1.27 1.27)) hide)
-    )
-    (property "Datasheet" "" (id 3) (at 163.83 57.15 0)
-      (effects (font (size 1.27 1.27)) hide)
-    )
-    (pin "1")
   )
   (symbol (lib_id "KD_Capacitor:C_0805_DNP") (at 152.4 69.85 0)
@@
     (pin "1")
   )
-  (symbol (lib_id "power:+3V3") (at 125.73 81.28 0)
+  (symbol (lib_id "power:+5V") (at 125.73 81.28 0)
     (in_bom yes) (on_board yes) (fields_autoplaced)
     (property "Reference" "#PWR?" (id 0) (at 125.73 85.09 0)
       (effects (font (size 1.27 1.27)) hide)
     )
-    (property "Value" "+3V3" (id 1) (at 125.73 76.2 0))
+    (property "Value" "+5V" (id 1) (at 125.73 76.2 0))
     (property "Footprint" "" (id 2) (at 125.73 81.28 0)
       (effects (font (size 1.27 1.27)) hide)
@@
     (pin "2")
   )
+  (symbol (lib_id "power:+5V") (at 163.83 57.15 0)
+    (in_bom yes) (on_board yes) (fields_autoplaced)
+    (property "Reference" "#PWR?" (id 0) (at 163.83 60.96 0)
+      (effects (font (size 1.27 1.27)) hide)
+    )
+    (property "Value" "+5V" (id 1) (at 163.83 52.07 0))
+    (property "Footprint" "" (id 2) (at 163.83 57.15 0)
+      (effects (font (size 1.27 1.27)) hide)
+    )
+    (property "Datasheet" "" (id 3) (at 163.83 57.15 0)
+      (effects (font (size 1.27 1.27)) hide)
+    )
+    (pin "1")
+  )
 )

Commit message: rikki
Parts:
- C19: renamed from C?; value C_0603_100n_X7R_50V -> C_0603_100n_X7R_100V; symbol KD_Capacitor:C_0603_100n_X7R_50V -> KD_Capacitor:C_0603_100n_X7R_100V; MFG_PartNo CL10B104KB8NNWC -> CL10B104KC8NNNC; Manufacturer Samsung -> Samsung Electro-Mechanics; Price 0.01 -> 0.03; Supplier_PartNo 1276-1935-1-ND -> 1276-6807-1-ND
- C20: renamed from C?; value C_0805_1u_X7R_25V -> C_0805_DNP
- R26, R27: renamed from R?; footprint KD_Resistor:R_0603_1608Metric -> KD_Resistor:RESC1608X55N
- U4: renamed from U?; footprint KD_Package_SO:SOIC127P600X200-16N -> KD_Package_SO:SOIC127P640X200-16N
Changed lines of the file:
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@@
   (title_block
     (title "Gear Display Board")
-    (date "2022-08-07")
+    (date "2022-08-13")
     (rev "1.0")
     (company "Kallio Designs Oy")
     (comment 1 "Teemu Latonen")
-    (comment 2 "ASSEMBLY_PN")
-    (comment 3 "PCB_PN")
+    (comment 2 "000064")
+    (comment 3 "000065")
   )
   (bus_alias "I2C" (members "SDA" "SCL"))
-  (bus_alias "SPI" (members "MISO" "MOSI" "SCLK"))
+  (bus_alias "SPI" (members "MISO" "MOSI" "SCLK" "CS"))
   (junction (at 163.83 63.5) (diameter 0) (color 0 0 0 0)
   )
@@
     (effects (font (size 1.27 1.27)) (justify right))
   )
-  (symbol (lib_id "KD_Capacitor:C_0805_DNP") (at 152.4 69.85 0)
+  (symbol (lib_id "KD_Capacitor:C_0805_DNP") (at 152.4 69.85 0) (unit 1)
     (in_bom yes) (on_board yes)
-    (property "Reference" "C?" (id 0) (at 154.94 68.58 0)
-      (effects (font (size 1.27 1.27)) (justify left))
-    )
-    (property "Value" "C_0805_1u_X7R_25V" (id 1) (at 139.7 38.1 0)
+    (property "Reference" "C20" (id 0) (at 154.94 68.58 0)
+      (effects (font (size 1.27 1.27)) (justify left))
+    )
+    (property "Value" "C_0805_DNP" (id 1) (at 139.7 38.1 0)
       (effects (font (size 1.27 1.27)) (justify left) hide)
     )
@@
     (pin "2")
   )
-  (symbol (lib_id "KD_IC_Buffer_Driver_Interface:Shift_register_OC_8bit_STPIC6D595MTR") (at 163.83 105.41 0)
-    (in_bom yes) (on_board yes) (fields_autoplaced)
-    (property "Reference" "U?" (id 0) (at 165.8494 87.63 0)
+  (symbol (lib_id "KD_IC_Buffer_Driver_Interface:Shift_register_OC_8bit_STPIC6D595MTR") (at 163.83 105.41 0) (unit 1)
+    (in_bom yes) (on_board yes) (fields_autoplaced)
+    (property "Reference" "U4" (id 0) (at 165.8494 87.63 0)
       (effects (font (size 1.27 1.27)) (justify left))
     )
@@
       (effects (font (size 1.27 1.27)) (justify left) hide)
     )
-    (property "Footprint" "KD_Package_SO:SOIC127P600X200-16N" (id 2) (at 146.05 60.96 0)
+    (property "Footprint" "KD_Package_SO:SOIC127P640X200-16N" (id 2) (at 146.05 60.96 0)
       (effects (font (size 1.27 1.27)) (justify left) hide)
     )
@@
     (pin "9")
   )
-  (symbol (lib_id "power:GND") (at 161.29 129.54 0)
-    (in_bom yes) (on_board yes) (fields_autoplaced)
-    (property "Reference" "#PWR?" (id 0) (at 161.29 135.89 0)
+  (symbol (lib_id "power:GND") (at 161.29 129.54 0) (unit 1)
+    (in_bom yes) (on_board yes) (fields_autoplaced)
+    (property "Reference" "#PWR0127" (id 0) (at 161.29 135.89 0)
       (effects (font (size 1.27 1.27)) hide)
     )
@@
     (pin "1")
   )
-  (symbol (lib_id "power:+5V") (at 125.73 81.28 0)
-    (in_bom yes) (on_board yes) (fields_autoplaced)
-    (property "Reference" "#PWR?" (id 0) (at 125.73 85.09 0)
+  (symbol (lib_id "power:+5V") (at 125.73 81.28 0) (unit 1)
+    (in_bom yes) (on_board yes) (fields_autoplaced)
+    (property "Reference" "#PWR0130" (id 0) (at 125.73 85.09 0)
       (effects (font (size 1.27 1.27)) hide)
     )
@@
     (pin "1")
   )
-  (symbol (lib_id "KD_Resistor:R_0603_22k_1%") (at 133.35 118.11 0)
-    (in_bom yes) (on_board yes) (fields_autoplaced)
-    (property "Reference" "R?" (id 0) (at 135.89 116.8399 0)
+  (symbol (lib_id "KD_Resistor:R_0603_22k_1%") (at 133.35 118.11 0) (unit 1)
+    (in_bom yes) (on_board yes) (fields_autoplaced)
+    (property "Reference" "R27" (id 0) (at 135.89 116.8399 0)
       (effects (font (size 1.27 1.27)) (justify left))
     )
@@
       (effects (font (size 1.27 1.27)) (justify left) hide)
     )
-    (property "Footprint" "KD_Resistor:R_0603_1608Metric" (id 2) (at 120.65 104.14 0)
+    (property "Footprint" "KD_Resistor:RESC1608X55N" (id 2) (at 120.65 104.14 0)
       (effects (font (size 1.27 1.27)) (justify left) hide)
     )
@@
     (pin "2")
   )
-  (symbol (lib_id "power:GND") (at 133.35 130.81 0)
-    (in_bom yes) (on_board yes) (fields_autoplaced)
-    (property "Reference" "#PWR?" (id 0) (at 133.35 137.16 0)
+  (symbol (lib_id "power:GND") (at 133.35 130.81 0) (unit 1)
+    (in_bom yes) (on_board yes) (fields_autoplaced)
+    (property "Reference" "#PWR0128" (id 0) (at 133.35 137.16 0)
       (effects (font (size 1.27 1.27)) hide)
     )
@@
     (pin "1")
   )
-  (symbol (lib_id "KD_Capacitor:C_0603_100n_X7R_50V") (at 137.16 69.85 0)
+  (symbol (lib_id "KD_Capacitor:C_0603_100n_X7R_100V") (at 137.16 69.85 0) (unit 1)
     (in_bom yes) (on_board yes)
-    (property "Reference" "C?" (id 0) (at 139.7 68.58 0)
-      (effects (font (size 1.27 1.27)) (justify left))
-    )
-    (property "Value" "C_0603_100n_X7R_50V" (id 1) (at 124.46 38.1 0)
+    (property "Reference" "C19" (id 0) (at 139.7 68.58 0)
+      (effects (font (size 1.27 1.27)) (justify left))
+    )
+    (property "Value" "C_0603_100n_X7R_100V" (id 1) (at 124.46 38.1 0)
       (effects (font (size 1.27 1.27)) (justify left) hide)
     )
@@
       (effects (font (size 1.27 1.27)) (justify left) hide)
     )
-    (property "Datasheet" "http://www.samsungsem.com/kr/support/product-search/mlcc/CL10B104KB8NNWC.jsp" (id 3) (at 124.46 58.42 0)
+    (property "Datasheet" "https://media.digikey.com/pdf/Data%20Sheets/Samsung%20PDFs/CL10B104KC8NNNC_Spec.pdf" (id 3) (at 124.46 58.42 0)
       (effects (font (size 1.27 1.27)) (justify left) hide)
     )
@@
       (effects (font (size 1.27 1.27)) (justify left))
     )
-    (property "Manufacturer" "Samsung" (id 5) (at 124.46 40.64 0)
-      (effects (font (size 1.27 1.27)) (justify left) hide)
-    )
-    (property "MFG_PartNo" "CL10B104KB8NNWC" (id 6) (at 124.46 43.18 0)
+    (property "Manufacturer" "Samsung Electro-Mechanics" (id 5) (at 124.46 40.64 0)
+      (effects (font (size 1.27 1.27)) (justify left) hide)
+    )
+    (property "MFG_PartNo" "CL10B104KC8NNNC" (id 6) (at 124.46 43.18 0)
       (effects (font (size 1.27 1.27)) (justify left) hide)
     )
@@
       (effects (font (size 1.27 1.27)) (justify left) hide)
     )
-    (property "Supplier_PartNo" "1276-1935-1-ND" (id 8) (at 124.46 48.26 0)
+    (property "Supplier_PartNo" "1276-6807-1-ND" (id 8) (at 124.46 48.26 0)
       (effects (font (size 1.27 1.27)) (justify left) hide)
     )
@@
       (effects (font (size 1.27 1.27)) (justify left) hide)
     )
-    (property "Price" "0.01" (id 10) (at 124.46 53.34 0)
+    (property "Price" "0.03" (id 10) (at 124.46 53.34 0)
       (effects (font (size 1.27 1.27)) (justify left) hide)
     )
@@
     (pin "2")
   )
-  (symbol (lib_id "power:GND") (at 152.4 78.74 0)
-    (in_bom yes) (on_board yes) (fields_autoplaced)
-    (property "Reference" "#PWR?" (id 0) (at 152.4 85.09 0)
+  (symbol (lib_id "power:GND") (at 152.4 78.74 0) (unit 1)
+    (in_bom yes) (on_board yes) (fields_autoplaced)
+    (property "Reference" "#PWR0129" (id 0) (at 152.4 85.09 0)
       (effects (font (size 1.27 1.27)) hide)
     )
@@
     (pin "1")
   )
-  (symbol (lib_id "KD_Resistor:R_0603_22k_1%") (at 125.73 87.63 0)
-    (in_bom yes) (on_board yes) (fields_autoplaced)
-    (property "Reference" "R?" (id 0) (at 128.27 86.3599 0)
+  (symbol (lib_id "KD_Resistor:R_0603_22k_1%") (at 125.73 87.63 0) (unit 1)
+    (in_bom yes) (on_board yes) (fields_autoplaced)
+    (property "Reference" "R26" (id 0) (at 128.27 86.3599 0)
       (effects (font (size 1.27 1.27)) (justify left))
     )
@@
       (effects (font (size 1.27 1.27)) (justify left) hide)
     )
-    (property "Footprint" "KD_Resistor:R_0603_1608Metric" (id 2) (at 113.03 73.66 0)
+    (property "Footprint" "KD_Resistor:RESC1608X55N" (id 2) (at 113.03 73.66 0)
       (effects (font (size 1.27 1.27)) (justify left) hide)
     )
@@
     (pin "2")
   )
-  (symbol (lib_id "power:+5V") (at 163.83 57.15 0)
-    (in_bom yes) (on_board yes) (fields_autoplaced)
-    (property "Reference" "#PWR?" (id 0) (at 163.83 60.96 0)
-      (effects (font (size 1.27 1.27)) hide)
-    )
+  (symbol (lib_id "power:+5V") (at 163.83 57.15 0) (unit 1)
+    (in_bom yes) (on_board yes) (fields_autoplaced)
+    (property "Reference" "#PWR0131" (id 0) (at 163.83 60.96 0)
+      (effects (font (size 1.27 1.27)) hide)
+    )

Commit message: PSU and LED powering changed
Parts:
- C19: footprint KD_Capacitor:C_0603_1608Metric -> KD_Capacitor:CAPC1608X90N
- C20: footprint KD_Capacitor:C_0805_2012Metric_DNP -> KD_Capacitor:CAPC2012X135N_DNP
Changed lines of the file:
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@@
       (effects (font (size 1.27 1.27)) (justify left) hide)
     )
-    (property "Footprint" "KD_Capacitor:C_0805_2012Metric_DNP" (id 2) (at 139.7 55.88 0)
+    (property "Footprint" "KD_Capacitor:CAPC2012X135N_DNP" (id 2) (at 139.7 55.88 0)
       (effects (font (size 1.27 1.27)) (justify left) hide)
     )
@@
       (effects (font (size 1.27 1.27)) (justify left) hide)
     )
-    (property "Footprint" "KD_Capacitor:C_0603_1608Metric" (id 2) (at 124.46 55.88 0)
+    (property "Footprint" "KD_Capacitor:CAPC1608X90N" (id 2) (at 124.46 55.88 0)
       (effects (font (size 1.27 1.27)) (justify left) hide)
     )
