File: gear-display/PCB/GDBM/led_driver.kicad_sch (KiCad schematic)
At the start: 5 parts, among them U4 Shift_register_OC_8bit_STPIC6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

Commit message: Layout
Parts:
- C19: value C_0603_100n_X7R_100V -> 100n
- C20: value C_0805_DNP -> 0805
Changed lines of the file:
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@@
     (comment 3 "000065")
   )
+  (bus_alias "I2C" (members "SDA" "SCL"))
   (bus_alias "SPI" (members "MISO" "MOSI" "SCLK" "CS"))
-  (bus_alias "I2C" (members "SDA" "SCL"))
   (junction (at 163.83 63.5) (diameter 0) (color 0 0 0 0)
   )
@@
       (effects (font (size 1.27 1.27)) (justify left))
     )
-    (property "Value" "C_0805_DNP" (at 139.7 38.1 0)
+    (property "Value" "0805" (at 139.7 38.1 0)
       (effects (font (size 1.27 1.27)) (justify left) hide)
     )
@@
       (effects (font (size 1.27 1.27)) (justify left) hide)
     )
-    (property "Datasheet" "https://api.kemet.com/component-edge/download/datasheet/CBR08C279B5GAC.pdf" (at 139.7 58.42 0)
+    (property "Datasheet" "datasheet" (at 139.7 58.42 0)
       (effects (font (size 1.27 1.27)) (justify left) hide)
     )
@@
       (effects (font (size 1.27 1.27)) (justify left))
     )
-    (property "Value" "C_0603_100n_X7R_100V" (at 124.46 38.1 0)
-      (effects (font (size 1.27 1.27)) (justify left) hide)
-    )
+    (property "Value" "100n" (at 124.46 38.1 0)
+      (effects (font (size 1.27 1.27)) (justify left) hide)
+    )
