File: gear-display/PCB/GDBM/GDBM.kicad_pcb (KiCad board)
At the start: 2 copper layers, 96 x 87 mm, 101 parts, among them J1 Con_Screw_1x04_691313510004, J2 Con_Screw_1x04_691313510004, J3 DC_2.1_5.5_54-00286, J4 Con_Screw_1x04_691313510004, J5 Con_Screw_1x04_691313510004, J6 Con_Screw_1x04_691313510004, J7 Con_Screw_1x04_691313510004, J8 USB_B_V_Adam_USB-B-S-VT, M1 Knob_6mm_BL_RED_CLIFF_CL17084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, Q1 PMOS_30V_4A1_SIL3407-TP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

Commit message: documentation update
Other:
- board text added: "Teemu Latonen | KD Oy | 000065 Rev 3.0"
- board text removed: "Teemu Latonen | KD Oy | 000065 Rev 2.0"
Changed lines of the file:
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@@
   (title_block
     (title "Gear Display Board")
-    (date "2023-01-05")
-    (rev "2.0")
+    (date "2023-04-06")
+    (rev "3.0")
     (company "Kallio Designs Oy")
     (comment 1 "Teemu Latonen")
@@
   (gr_rect (start 18.2 39.2) (end 35.2 41.2)
     (stroke (width 0.1) (type solid)) (fill none) (layer "F.Fab"))
-  (gr_text "Teemu Latonen | KD Oy | 000065 Rev 2.0" (at 130.15 155) (layer "B.Cu")
+  (gr_text "Teemu Latonen | KD Oy | 000065 Rev 3.0" (at 130.15 155) (layer "B.Cu")
     (effects (font (size 1.5 1.5) (thickness 0.3)) (justify mirror))
   )

Commit message: Revert "documentation update"
This reverts commit 76ec955dce09cc544308a8dd0d1d241e10a4399a.
Other:
- board text added: "Teemu Latonen | KD Oy | 000065 Rev 2.0"
- board text removed: "Teemu Latonen | KD Oy | 000065 Rev 3.0"
Changed lines of the file:
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@@
   (title_block
     (title "Gear Display Board")
-    (date "2023-04-06")
-    (rev "3.0")
+    (date "2023-01-05")
+    (rev "2.0")
     (company "Kallio Designs Oy")
     (comment 1 "Teemu Latonen")
@@
   (gr_rect (start 18.2 39.2) (end 35.2 41.2)
     (stroke (width 0.1) (type solid)) (fill none) (layer "F.Fab"))
-  (gr_text "Teemu Latonen | KD Oy | 000065 Rev 3.0" (at 130.15 155) (layer "B.Cu")
+  (gr_text "Teemu Latonen | KD Oy | 000065 Rev 2.0" (at 130.15 155) (layer "B.Cu")
     (effects (font (size 1.5 1.5) (thickness 0.3)) (justify mirror))
   )

Commit message: R33 value change
Parts:
- added R34: R_0402_4700_1%, KD_Resistor:RESC1005X40N, B.Cu at (129.8, 98.0)
- R33: value R_0805_1200_5% -> R_0805_110_5%
Connections:
- Q1 pad 1: +12V -> /7-Segment Display/12V_PWM
- Q1 pad 2: +12V -> /7-Segment Display/12V_PWM
- Q1 pad 4: /7-Segment Display/12V_PWM -> +12V
- Q1 pad 5: +12V -> /7-Segment Display/12V_PWM
- Q1 pad 6: +12V -> /7-Segment Display/12V_PWM
- U2 pad 41: /7-Segment Display/PWM -> /MCU/A5(D23)
- U4 pad 11: /7-Segment Display/e -> /7-Segment Display/d
- U4 pad 12: /7-Segment Display/f -> /7-Segment Display/c
- U4 pad 13: /7-Segment Display/g -> /7-Segment Display/b
- U4 pad 14: /7-Segment Display/dp -> /7-Segment Display/a
- U4 pad 3: /7-Segment Display/a -> /7-Segment Display/dp
- U4 pad 4: /7-Segment Display/b -> /7-Segment Display/g
- U4 pad 5: /7-Segment Display/c -> /7-Segment Display/f
- U4 pad 6: /7-Segment Display/d -> /7-Segment Display/e
Routing:
- net /7-Segment Display/12V_PWM: track 79.2 -> 84.0 mm
- net +12V: track 52.3 -> 47.5 mm

Commit message: documentation
Parts:
- moved R34 1.27 mm to (130.0, 96.8)
Connections:
- U4 pad 11: /7-Segment Display/d -> /7-Segment Display/e
- U4 pad 12: /7-Segment Display/c -> /7-Segment Display/f
- U4 pad 13: /7-Segment Display/b -> /7-Segment Display/g
- U4 pad 14: /7-Segment Display/a -> /7-Segment Display/dp
- U4 pad 3: /7-Segment Display/dp -> /7-Segment Display/a
- U4 pad 4: /7-Segment Display/g -> /7-Segment Display/b
- U4 pad 5: /7-Segment Display/f -> /7-Segment Display/c
- U4 pad 6: /7-Segment Display/e -> /7-Segment Display/d
Routing:
- net /MCU/A5(D23): track 0.00 -> 5.13 mm
- net /7-Segment Display/PWM: track 192.3 -> 189.4 mm
Other:
- board text added: "Teemu Latonen | KD Oy | 000065 Rev 3.0"
- board text removed: "Teemu Latonen | KD Oy | 000065 Rev 2.0"

Commit message: Layout
Parts:
- added C26: 10u, KD_Capacitor:CAPC3216X150N, B.Cu at (93.2, 93.4)
- C1, C12, C16, C17, C2, C25, C3: value C_1206_10u_X5R_50V_automotive -> 10u
- C10, C8: value C_0603_33p_NP0_5%_100V -> 33p
- C11, C21, C7, C9: value C_0805_1u_X7R_25V -> 1u
- C13, C14, C18, C19, C4, C5, C6: value C_0603_100n_X7R_100V -> 100n
- C15, C20: value C_0805_DNP -> 0805
- C22: value C_0805_22u_X5R_10V -> 10u; footprint KD_Capacitor:CAPC2012X135N -> KD_Capacitor:CAPC3216X150N
- C23, C24: value C_0603_10n_X7R_100V -> 10n
- D3: footprint KD_Diode:DIOC1608X70N -> KD_Diode:LEDM1608X70M
- FD1, FD2, FD3, FD4, FD5, FD6: value Fiducial_0.5mm -> Fiducial 0.5 mm
- H1, H3, H4, H5, H6: value NPTH_3.2_M3_Clearance -> NPTH 3.2 M3 Clearance
- J1, J2, J4, J5, J6, J7: value Con_Screw_1x04_691313510004 -> 1x04
- J8: value USB_B_V_Adam_USB-B-S-VT -> USB Mini B
- R1, R22: value R_0805_DNP -> DNP
- R20, R21, R23, R24, R25: value R_0805_0_automotive -> 0
- R28: value Pot_V_10k_CUI_PT01-D120K2-B103 -> PT01-D225D-A503
- R31, R32, R34: value R_0402_4700_1% -> 4k7
- U3: value Gate_Driver_MCP1401T-E-OT -> MCP1401
- X3: value CON_GND_Probe_Hook -> GND Hook
- Y1: value Crystal_16M_AS-16.000-18-SMD-TR -> 16 MHz
- moved C15 9.22 mm to (109.5, 136.5), turned to 0 degrees
- moved C14 1.14 mm to (104.5, 144.5), turned to 0 degrees
Connections:
- D7 pad 1: Net-(D7-K) -> Net-(D6-A)
- D7 pad 2: Net-(D6-K) -> Net-(D7-A)
- R28 pad 1: Net-(D7-K) -> Net-(D7-A)
- R28 pad 3: Net-(D6-A) -> Net-(D6-K)
- R33 pad 2: Net-(D6-K) -> Net-(D6-A)
- U5 pad 7: Net-(D6-K) -> Net-(D6-A)
Routing:
- net Net-(D7-K): track 27.9 -> 0.00 mm
- net Net-(D7-A): track 0.00 -> 24.9 mm
- net /7-Segment Display/PWM: track 189.4 -> 192.4 mm
- net Net-(D6-A): track 13.9 -> 13.4 mm
- net +12V: track 47.5 -> 48.0 mm
Other:
- board text added: "Teemu Latonen | KD Oy | 000065 Rev 4.0"
- board text removed: "Teemu Latonen | KD Oy | 000065 Rev 3.0"
