File: gear-display/PCB/GDBM/7seg_display.kicad_sch (KiCad schematic)
At the start: 15 parts, among them Q1 PMOS_30V_4A1_SIL3407-TP, U3 Gate_Driver_MCP1401T-E-OT

Commit message: Layout
Parts:
- C14: value C_0603_100n_X7R_100V -> 100n
- C15: value C_0805_DNP -> 0805
- U3: value Gate_Driver_MCP1401T-E-OT -> MCP1401
Changed lines of the file:
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@@
       (effects (font (size 1.27 1.27)) (justify left))
     )
-    (property "Value" "C_0603_100n_X7R_100V" (at 88.9 3.81 0)
+    (property "Value" "100n" (at 88.9 3.81 0)
       (effects (font (size 1.27 1.27)) (justify left) hide)
     )
@@
       (effects (font (size 1.27 1.27)) (justify left))
     )
-    (property "Value" "C_0805_DNP" (at 104.14 3.81 0)
+    (property "Value" "0805" (at 104.14 3.81 0)
       (effects (font (size 1.27 1.27)) (justify left) hide)
     )
@@
       (effects (font (size 1.27 1.27)) (justify left) hide)
     )
-    (property "Datasheet" "https://api.kemet.com/component-edge/download/datasheet/CBR08C279B5GAC.pdf" (at 104.14 24.13 0)
+    (property "Datasheet" "datasheet" (at 104.14 24.13 0)
       (effects (font (size 1.27 1.27)) (justify left) hide)
     )
@@
       (effects (font (size 1.27 1.27)))
     )
-    (property "Value" "Gate_Driver_MCP1401T-E-OT" (at 113.03 15.24 0)
-      (effects (font (size 1.27 1.27)) (justify left) hide)
-    )
+    (property "Value" "MCP1401" (at 113.03 15.24 0)
+      (effects (font (size 1.27 1.27)) (justify left) hide)
+    )

Commit message: Documentation update
Other:
- note removed: "Pitäiskö vaihtaa MCP1402, jotta säätö olis 0-50 %"
Changed lines of the file:
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@@
     (stroke (width 0) (type default))
-  )
-  (text "Pitäiskö vaihtaa MCP1402, jotta säätö olis 0-50 %" (at 95.25 83.82 0)
-    (effects (font (size 2 2)) (justify left bottom))
   )
   (hierarchical_label "PWM" (shape input) (at 73.66 59.69 180) (fields_autoplaced)
