File: gear-display/PCB/GDBM/main.kicad_sch (KiCad schematic)
At the start: 19 parts, among them U2 ATmega32U4-AU, X1 Programming_AVR_ISP_Staggered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, X2 CON_1x04_TH_staggered, Y1 Crystal_16M_AS-16.000-18-SMD-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

Commit message: Layout
Parts:
- C10, C8: value C_0603_33p_NP0_5%_100V -> 33p
- C11, C7, C9: value C_0805_1u_X7R_25V -> 1u; Manufacturer Kemet -> Samsung Electro-Mechanics
- C6: value C_0603_100n_X7R_100V -> 100n
- D3: footprint KD_Diode:DIOC1608X70N -> KD_Diode:LEDM1608X70M
- R1: value R_0805_DNP -> DNP
- Y1: value Crystal_16M_AS-16.000-18-SMD-TR -> 16 MHz
