File: gear-display/PCB/GDBM/mechanical.kicad_sch (KiCad schematic)
At the start: 13 parts, among them X3 CON_GND_Probe_Hook

Commit message: Layout
Parts:
- FD1, FD2, FD3, FD4, FD5, FD6: value Fiducial_0.5mm -> Fiducial 0.5 mm
- H1, H3, H4, H5, H6: value NPTH_3.2_M3_Clearance -> NPTH 3.2 M3 Clearance
- X3: value CON_GND_Probe_Hook -> GND Hook
Changed lines of the file:
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@@
       (effects (font (size 1.27 1.27)) (justify left))
     )
-    (property "Value" "NPTH_3.2_M3_Clearance" (at 50.8 38.1 0)
+    (property "Value" "NPTH 3.2 M3 Clearance" (at 50.8 38.1 0)
       (effects (font (size 1.27 1.27)) (justify left) hide)
     )
@@
       (effects (font (size 1.27 1.27)) (justify left))
     )
-    (property "Value" "NPTH_3.2_M3_Clearance" (at 50.8 25.4 0)
+    (property "Value" "NPTH 3.2 M3 Clearance" (at 50.8 25.4 0)
       (effects (font (size 1.27 1.27)) (justify left) hide)
     )
@@
       (effects (font (size 1.27 1.27)) (justify left))
     )
-    (property "Value" "Fiducial_0.5mm" (at 25.4 12.7 0)
+    (property "Value" "Fiducial 0.5 mm" (at 25.4 12.7 0)
       (effects (font (size 1.27 1.27)) (justify left) hide)
     )
@@
       (effects (font (size 1.27 1.27)) (justify left))
     )
-    (property "Value" "CON_GND_Probe_Hook" (at 111.76 30.48 0)
+    (property "Value" "GND Hook" (at 111.76 30.48 0)
       (effects (font (size 1.27 1.27)) (justify left) hide)
     )
@@
       (effects (font (size 1.27 1.27)) (justify left))
     )
-    (property "Value" "NPTH_3.2_M3_Clearance" (at 50.8 31.75 0)
+    (property "Value" "NPTH 3.2 M3 Clearance" (at 50.8 31.75 0)
       (effects (font (size 1.27 1.27)) (justify left) hide)
     )
@@
       (effects (font (size 1.27 1.27)) (justify left))
     )
-    (property "Value" "Fiducial_0.5mm" (at 25.4 25.4 0)
+    (property "Value" "Fiducial 0.5 mm" (at 25.4 25.4 0)
       (effects (font (size 1.27 1.27)) (justify left) hide)
     )
@@
       (effects (font (size 1.27 1.27)) (justify left))
     )
-    (property "Value" "NPTH_3.2_M3_Clearance" (at 50.8 19.05 0)
+    (property "Value" "NPTH 3.2 M3 Clearance" (at 50.8 19.05 0)
       (effects (font (size 1.27 1.27)) (justify left) hide)
     )
@@
       (effects (font (size 1.27 1.27)) (justify left))
     )
-    (property "Value" "Fiducial_0.5mm" (at 25.4 19.05 0)
+    (property "Value" "Fiducial 0.5 mm" (at 25.4 19.05 0)
       (effects (font (size 1.27 1.27)) (justify left) hide)
     )
@@
       (effects (font (size 1.27 1.27)) (justify left))
     )
-    (property "Value" "NPTH_3.2_M3_Clearance" (at 50.8 6.35 0)
+    (property "Value" "NPTH 3.2 M3 Clearance" (at 50.8 6.35 0)
       (effects (font (size 1.27 1.27)) (justify left) hide)
     )
@@
       (effects (font (size 1.27 1.27)) (justify left) hide)
     )
+    (property "Sim.Enable" "0" (at 126.492 26.67 0)
+      (effects (font (size 1.27 1.27)) hide)
+    )
     (instances
       (project "GDBM"
@@
       (effects (font (size 1.27 1.27)) (justify left))
     )
-    (property "Value" "Fiducial_0.5mm" (at 25.4 38.1 0)
+    (property "Value" "Fiducial 0.5 mm" (at 25.4 38.1 0)
       (effects (font (size 1.27 1.27)) (justify left) hide)
     )
@@
       (effects (font (size 1.27 1.27)) (justify left))
     )
-    (property "Value" "Fiducial_0.5mm" (at 25.4 6.35 0)
+    (property "Value" "Fiducial 0.5 mm" (at 25.4 6.35 0)
       (effects (font (size 1.27 1.27)) (justify left) hide)
     )
@@
       (effects (font (size 1.27 1.27)) (justify left))
     )
-    (property "Value" "Fiducial_0.5mm" (at 25.4 31.75 0)
-      (effects (font (size 1.27 1.27)) (justify left) hide)
-    )
+    (property "Value" "Fiducial 0.5 mm" (at 25.4 31.75 0)
+      (effects (font (size 1.27 1.27)) (justify left) hide)
+    )
